Commit message: fix: 车体高度修正+轮子位置修正实现Gazebo内真实移动

File: src/embobot_description/xacro/base.xacro (robot description, xacro)
@@ -6,5 +6,5 @@
     <parent link="base_footprint"/>
     <child link="base_link"/>
-    <origin xyz="0.0 0.0 ${wheel_radius}" rpy="0 0 0"/>
+    <origin xyz="0.0 0.0 ${base_height/2 + wheel_radius}" rpy="0 0 0"/>
   </joint>
   <!-- 底盘主体 -->

File: src/embobot_description/xacro/gazebo.xacro (robot description, xacro)
@@ -22,14 +22,14 @@
   <!-- ③  驱动轮摩擦力（较大，保证抓地力）-->
   <gazebo reference="left_wheel_link">
-    <mu1>1.0</mu1>
-    <mu2>0.5</mu2>
-    <kp>500000.0</kp>
-    <kd>10.0</kd>
+    <mu1>10.0</mu1>
+    <mu2>5.0</mu2>
+    <kp>1000000.0</kp>
+    <kd>100.0</kd>
   </gazebo>
   <gazebo reference="right_wheel_link">
-    <mu1>1.0</mu1>
-    <mu2>0.5</mu2>
-    <kp>500000.0</kp>
-    <kd>10.0</kd>
+    <mu1>10.0</mu1>
+    <mu2>5.0</mu2>
+    <kp>1000000.0</kp>
+    <kd>100.0</kd>
   </gazebo>
   <!-- ④  激光雷达传感器插件（Gazebo Harmonic 语法）-->

File: src/embobot_description/xacro/macros.xacro (robot description, xacro)
@@ -72,5 +72,5 @@
       <parent link="base_link"/>
       <child link="${name}_wheel_link"/>
-      <origin xyz="0 ${y_offset} 0" rpy="0 0 0"/>
+      <origin xyz="0 ${y_offset} ${-base_height/2}" rpy="0 0 0"/>
       <axis xyz="0 1 0"/>
     </joint>

Commit message: fix: 修正万向轮接地并记录雷达假墙排查

File: src/embobot_description/xacro/base.xacro (robot description, xacro)
@@ -21,5 +21,5 @@
     <xacro:cylinder_inertia m="${base_mass}" r="${base_radius}" h="${base_height}"/>
   </link>
-  <!-- 万向轮 -->
+  <!-- 前万向轮 -->
   <link name="caster_link">
     <visual>
@@ -35,5 +35,21 @@
     <parent link="base_link"/>
     <child link="caster_link"/>
-    <origin xyz="${caster_x} 0.0 ${-(base_height/2 - caster_radius)}" rpy="0 0 0"/>
+    <origin xyz="${caster_x} 0.0 ${caster_radius - (base_height/2 + wheel_radius)}" rpy="0 0 0"/>
+  </joint>
+  <!-- 后万向轮：与前万向轮形成前后支撑，减少加减速时车体俯仰 -->
+  <link name="rear_caster_link">
+    <visual>
+      <geometry><sphere radius="${caster_radius}"/></geometry>
+      <material name="light_gray"/>
+    </visual>
+    <collision>
+      <geometry><sphere radius="${caster_radius}"/></geometry>
+    </collision>
+    <xacro:sphere_inertia m="0.05" r="${caster_radius}"/>
+  </link>
+  <joint name="rear_caster_joint" type="fixed">
+    <parent link="base_link"/>
+    <child link="rear_caster_link"/>
+    <origin xyz="${-caster_x} 0.0 ${caster_radius - (base_height/2 + wheel_radius)}" rpy="0 0 0"/>
   </joint>
 </robot>

File: src/embobot_description/xacro/gazebo.xacro (robot description, xacro)
@@ -16,4 +16,9 @@
   <!-- ②  万向轮摩擦力（设为极小，让它可以自由滑动）-->
   <gazebo reference="caster_link">
+    <mu1>0.001</mu1>
+    <mu2>0.001</mu2>
+    <material>Gazebo/Grey</material>
+  </gazebo>
+  <gazebo reference="rear_caster_link">
     <mu1>0.001</mu1>
     <mu2>0.001</mu2>
